File: Hardware/WirelessJLink_V3S.kicad_pcb (KiCad board)
At the start: 4 copper layers, 39 x 40.5 mm, 147 parts, among them J1 Micro_SD_Card, J2 USB_C_Receptacle_USB2.0, J3 USB_C_Receptacle_USB2.0, J4 JLink_Upload, J5 JLINK_OUT, J6 24V_IN, Q1 S8050, SW1 海龟, U1 V831, U3 RS3236, U4 CH343P, U5 STM32F103CBT6, U6 W25Q128, U7 RTL8723BS, U8 RY8411, Y2 24MHz, Y3 8MHz

Commit message: V2 sch & layout Half Cplt
Parts:
- removed C2: 10nF, Capacitor_SMD:C_0603_1608Metric
- removed C36, C69: 100nF, Capacitor_SMD:C_0603_1608Metric
- removed C70: 100nF, Resistor_SMD:R_0603_1608Metric
- removed C71: 20pF, Resistor_SMD:R_0603_1608Metric
- removed C72, C73: 10uF, Capacitor_SMD:C_1206_3216Metric
- removed D3: K34, Diode_SMD:D_SMF
- removed F3: Fuse, Fuse:Fuse_1206_3216Metric
- removed J5: JLINK_OUT, Connector_Molex:Molex_PicoBlade_53261-0471_1x04-1MP_P1.25mm_Horizontal
- removed J6: 24V_IN, Connector_AMASS:AMASS_XT30PW-M_1x02_P2.50mm_Horizontal
- removed L4: 4.7uH, Inductor_SMD:L_Sunlord_SWPA252012S
- removed Q1: S8050, Package_TO_SOT_SMD:SOT-23
- removed R14, R15: 5.1K, Resistor_SMD:R_0603_1608Metric
- removed R16, R17: 33, Resistor_SMD:R_0603_1608Metric
- removed R2: 53.6K, Resistor_SMD:R_0603_1608Metric
- removed R20: 100R, Resistor_SMD:R_0603_1608Metric
- removed R21, R23, R33: 10K, Resistor_SMD:R_0603_1608Metric
- removed R22: 4.7K, Resistor_SMD:R_0603_1608Metric
- removed R26, R27, R3: 10k, Resistor_SMD:R_0603_1608Metric
- removed R28, R29: 33R, Resistor_SMD:R_0603_1608Metric
- removed R30: 1.5K, Resistor_SMD:R_0603_1608Metric
- removed R34: 36K, Resistor_SMD:R_0603_1608Metric
- removed R35, R41: 1K, Resistor_SMD:R_0603_1608Metric
- removed R36: 100, Resistor_SMD:R_0603_1608Metric
- removed R43: 33K, Resistor_SMD:R_0603_1608Metric
- removed SW1: 海龟, Button_Switch_SMD:SW_Push_1P1T_NO_CK_KMR2
- removed U3: RS3236, Package_TO_SOT_SMD:SOT-23-5
- removed U8: RY8411, Package_TO_SOT_SMD:SOT-23-6
- removed Y3: 8MHz, Crystal:Resonator_SMD_Murata_CSTxExxV-3Pin_3.0x1.1mm
- added R4: 33R, Resistor_SMD:R_0402_1005Metric, F.Cu at (223.3, 119.4)
- added Y1: 8MHz, Crystal:Resonator_SMD_Murata_CSTxExxV-3Pin_3.0x1.1mm, F.Cu at (213.3, 115.3)
- AE1: footprint 0_RM2024:IPXE4 -> RM2024:IPEX_1; moved to B.Cu
- C1, C14, C19, C26, C30, C32, C33, C34, C35, C40, C41, C42, C43, C44, C45, C53, C61, C63: footprint Capacitor_SMD:C_0603_1608Metric -> Capacitor_SMD:C_0402_1005Metric; moved to F.Cu
- C10, C11, C12, C4, C5: footprint Capacitor_SMD:C_1206_3216Metric -> Capacitor_SMD:C_0402_1005Metric; moved to B.Cu
- C13, C3, C6: footprint Capacitor_SMD:C_1206_3216Metric -> Capacitor_SMD:C_0402_1005Metric
- C15, C16, C17, C18, C22, C23, C27, C28, C29, C31, C37, C38, C39, C46, C47, C48, C49, C50, C51, C52, C54, C55, C56, C57, C58, C59, C60, C62, C64, C65, C66, C68: footprint Capacitor_SMD:C_0603_1608Metric -> Capacitor_SMD:C_0402_1005Metric
- C20, C21: value 20pF -> 100nF; footprint Capacitor_SMD:C_0603_1608Metric -> Capacitor_SMD:C_0402_1005Metric; moved to F.Cu
- C24: value 100nF -> 10uF; footprint Capacitor_SMD:C_0603_1608Metric -> Capacitor_SMD:C_0805_2012Metric
- C25, C67: footprint Capacitor_SMD:C_0603_1608Metric -> Capacitor_SMD:C_0402_1005Metric; moved to B.Cu
- C7, C8, C9, L1, L2, L3, R11, R8, U4, U5: moved to B.Cu
- D1, F2: moved to F.Cu
- D2: footprint LED_SMD:LED_0603_1608Metric -> LED_SMD:LED_0402_1005Metric
- D4: footprint LED_SMD:LED_0603_1608Metric -> LED_SMD:LED_0402_1005Metric; moved to F.Cu
- J1: footprint 0_RM2024:TF_Card_Short2 -> RM2024:TF_Card_Short2
- J2: footprint 0_RM2024:USB_C_Receptacle_HRO_TYPE-C-31-M-12_NO_HOLE -> Connector_USB:USB_C_Receptacle_GCT_USB4110; moved to F.Cu
- J3: value USB_C_Receptacle_USB2.0 -> JLink_Upload; footprint 0_RM2024:USB_C_Receptacle_HRO_TYPE-C-31-M-12_NO_HOLE -> Connector_Hirose:Hirose_DF13-04P-1.25DS_1x04_P1.25mm_Horizontal; moved to F.Cu
- J4: footprint Connector_Molex:Molex_PicoBlade_53048-0410_1x04_P1.25mm_Horizontal -> RM2024:1.25Upload
- R1, R40, R45, R5: footprint Resistor_SMD:R_0603_1608Metric -> Resistor_SMD:R_0402_1005Metric; moved to F.Cu
- R10: value 100K -> 10K; moved to B.Cu
- R12, R39, R42, R44, R46: footprint Resistor_SMD:R_0603_1608Metric -> Resistor_SMD:R_0402_1005Metric
- R13, R37, R38: footprint Resistor_SMD:R_0603_1608Metric -> Resistor_SMD:R_0402_1005Metric; moved to B.Cu
- R18: value 100K -> 33R; footprint Resistor_SMD:R_0603_1608Metric -> Resistor_SMD:R_0402_1005Metric; moved to F.Cu
- R19: value 10K -> 1K; footprint Resistor_SMD:R_0603_1608Metric -> Resistor_SMD:R_0402_1005Metric; moved to F.Cu
- R6: value 10K -> 200K; moved to B.Cu
- R7: value 200K -> 10K; moved to B.Cu
- R9: value 10K -> 100K; moved to B.Cu
- RN1, RN2: footprint Resistor_SMD:R_Array_Convex_4x0603 -> Resistor_SMD:R_Array_Convex_4x0402
- U2: footprint Package_DFN_QFN:HVQFN-24-1EP_4x4mm_P0.5mm_EP2.6x2.6mm_ThermalVias -> Package_DFN_QFN:HVQFN-24-1EP_4x4mm_P0.5mm_EP2.6x2.6mm; moved to B.Cu
- U6: value W25Q128 -> HT7133; footprint Package_SO:SOIC-8_5.23x5.23mm_P1.27mm -> Package_TO_SOT_SMD:SOT-23-3; moved to B.Cu
- U7: footprint 0_RM2024:RTL8723BS -> RM2024:RTL8723BS; moved to B.Cu
- moved AE1 71.8 mm to (212.4, 140.8), turned to 0 degrees
- moved C21 71.3 mm to (220.4, 123.3), turned to 0 degrees
- moved C22 70.5 mm to (220.4, 125.3), turned to 0 degrees
- moved C20 69.7 mm to (220.4, 121.3), turned to 0 degrees
- moved C3 68.8 mm to (205.4, 141.8), turned to 90 degrees
- moved J2 67.4 mm to (205.7, 151.6), turned to 0 degrees
- moved R13 65.3 mm to (207.9, 146.5)
- moved C19 64.6 mm to (220.4, 119.4), turned to 0 degrees
- moved C25 64.5 mm to (196.3, 147.0), turned to -90 degrees
- moved J3 61.7 mm to (203.6, 116.4), turned to 0 degrees
- moved C7 61.3 mm to (207.4, 143.7), turned to 90 degrees
- moved J4 60.9 mm to (221.8, 111.8), turned to 0 degrees
- moved R6 60.7 mm to (206.4, 143.7), turned to -90 degrees
- moved C13 60.3 mm to (196.3, 141.1), turned to 90 degrees
- moved C23 59.8 mm to (220.4, 127.3), turned to 0 degrees
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Connections:
- C10 pad 2: +1V2 -> +1V8
- C11 pad 2: +1V8 -> +1V2
- C13 pad 1: +24V -> GND
- C13 pad 2: GND -> +1V2
- C20 pad 1: GND -> +3V3
- C20 pad 2: /JLINK_DXIN -> GND
- C21 pad 1: GND -> +3V3
- C21 pad 2: /JLINK_DXOUT -> GND
- C25 pad 1: +3V3 -> GND
- C25 pad 2: GND -> +3V3
- C3 pad 1: +24V -> GND
- C3 pad 2: GND -> +1V8
- C7 pad 2: +1V2 -> +1V8
- C8 pad 2: +1V8 -> +1V2
- F2 pad 1: Net-(J5-Pin_1) -> Net-(J3-Pin_4)
- J4 pad 1: /ST_SWDIO -> +3V3
- J4 pad 2: /ST_SWCLK -> GND
- J4 pad 3: GND -> /ST_SWCLK
- J4 pad 4: +3V3 -> /ST_SWDIO
- L1 pad 2: +1V2 -> +1V8
- L2 pad 2: +1V8 -> +1V2
- R18 pad 1: +3V3 -> /T_JTCK_SWCLK
- R18 pad 2: Net-(U5-NRST) -> Net-(J3-Pin_2)
- R19 pad 1: Net-(U5-PC13) -> Net-(D2-A)
- R19 pad 2: GND -> +3V3
- R6 pad 1: +1V2 -> +1V8
- R7 pad 1: +1V8 -> +1V2
- U1 pad 110: /OTG_DM -> /JLINK_DM
- U1 pad 111: /OTG_DP -> /JLINK_DP
- U5 pad 10: Net-(U5-PA0) -> +3V3
- U5 pad 2: Net-(U5-PC13) -> GND
- U5 pad 25: /T_SWDIO_IN -> /T_JTMS_SWDIO
- U5 pad 3: Net-(U5-PC14) -> GND
- U5 pad 38: /JLINK_USB_RENUM -> unconnected-(U5-PA15-Pad38)
- U5 pad 39: Net-(U5-PB3) -> +3V3
- U5 pad 44: Net-(U5-BOOT0) -> GND
- U6 pad 1: /FLASH_CS -> GND
- U6 pad 2: /SPI0_MISO -> +3V0
- U6 pad 3: +3V3 -> +5V
Routing:
- net +3V3: track 100.3 -> 0.00 mm, vias 38 -> 0
- net +5V: track 81.2 -> 0.00 mm, vias 20 -> 0
- net +1V2: track 73.0 -> 0.00 mm, vias 20 -> 0
- net GND: track 53.5 -> 0.00 mm, vias 128 -> 0
- net +1V8: track 52.7 -> 0.00 mm, vias 13 -> 0
- net /JLINK_DM: track 37.7 -> 0.00 mm, vias 1 -> 0
- net /JLINK_DP: track 35.5 -> 0.00 mm, vias 1 -> 0
- net /WL_UART_RX: track 31.0 -> 0.00 mm, vias 2 -> 0
- net /OTG_DM: track 29.5 -> 0.00 mm, vias 3 -> 0
- net /WL_UART_TX: track 28.9 -> 0.00 mm
- net /OTG_DP: track 27.3 -> 0.00 mm, vias 3 -> 0
- net +3V0: track 24.0 -> 0.00 mm, vias 3 -> 0
- net VBUS: track 18.9 -> 0.00 mm, vias 9 -> 0
- net /UART_DP: track 17.1 -> 0.00 mm, vias 1 -> 0
- net /UART_DM: track 16.8 -> 0.00 mm, vias 1 -> 0
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- removed copper zone on F.Cu, net +1V2
- removed copper zone on In2.Cu, net +1V2
- removed copper zone on F.Cu, net +1V8
- removed copper zone on In2.Cu, net +1V8
- removed copper zone on B.Cu, net +24V
- removed copper zone on F.Cu, net +24V
- removed copper zone on F.Cu, net +3V3
- removed copper zone on In2.Cu, net +3V3
- removed copper zone on B.Cu, net +5V
- removed copper zone on F.Cu, net +5V
- removed copper zone on In2.Cu, net +5V
- removed copper zone on B.Cu, net GND
- removed copper zone on F.Cu, net GND
- removed copper zone on In1.Cu, net GND
- removed copper zone on B.Cu, net Net-(J5-Pin_1)
- removed copper zone on F.Cu, net Net-(J5-Pin_1)
- removed copper zone on F.Cu, net Net-(U2-LX1)
- removed copper zone on F.Cu, net Net-(U2-LX2)
- removed copper zone on F.Cu, net Net-(U2-LX3)
- removed copper zone on F.Cu, net Net-(U8-LX)
- removed copper zone on B.Cu, net VBUS
- removed copper zone on In2.Cu, net VBUS
Other:
- board size 39 x 40.5 mm -> 20.5 x 41.1 mm
- board text removed: "+ G C D"
- board text removed: "2.4G Wifi"
- board text removed: "FEL"
- board text removed: "ID"
- board text removed: "JLink"
- board text removed: "JLink/OTG"
- board text removed: "RM2025-ZZY"
- board text removed: "RTL8723"
- board text removed: "UART"
- board text removed: "V3S 无线烧录"
- board text removed: "全志 V3S Armhf"

Commit message: V2 Hardware Half Cplt
Parts:
- removed C20, C21, C22, C43, C47: 100nF, Capacitor_SMD:C_0402_1005Metric
- removed C60: 1uF, Capacitor_SMD:C_0402_1005Metric
- removed D4: LED, LED_SMD:LED_0402_1005Metric
- removed F2: 1A, Fuse:Fuse_1206_3216Metric
- removed R1: 1K, Resistor_SMD:R_0402_1005Metric
- added C2: 10uF, Capacitor_SMD:C_0402_1005Metric, B.Cu at (102.1, 123.7)
- added C36: 10uF, Capacitor_SMD:C_0402_1005Metric, B.Cu at (110.9, 130.6)
- added C69: 10uF, Capacitor_SMD:C_0402_1005Metric, B.Cu at (102.1, 129.6)
- added H1: M2, MountingHole:MountingHole_2.2mm_M2_DIN965, F.Cu at (102.5, 98.5)
- added H2: M2, MountingHole:MountingHole_2.2mm_M2_DIN965, F.Cu at (102.5, 135.8)
- added H3: M2, MountingHole:MountingHole_2.2mm_M2_DIN965, F.Cu at (121.7, 98.5)
- added H4: M2, MountingHole:MountingHole_2.2mm_M2_DIN965, F.Cu at (121.7, 135.8)
- added J5: TFT, RM2024:1.47TFT_12P, F.Cu at (112.3, 127.5)
- C1: value 100nF -> 10uF; moved to B.Cu
- C19, C23, C26, C27, C28, C35, C41, C42, C45, C61, J4, R45, R46, Y1, Y2: moved to B.Cu
- C51, C52, C62: moved to F.Cu
- moved C19 116.4 mm to (105.4, 101.2)
- moved R4 115.6 mm to (108.9, 102.8), turned to 90 degrees
- moved C30 113.6 mm to (109.9, 106.7), turned to -90 degrees
- moved Y1 109.0 mm to (104.9, 103.8), turned to -90 degrees
- moved C23 100.8 mm to (120.9, 111.2)
- moved J4 100.3 mm to (121.8, 103.3), turned to 180 degrees
- moved R18 99.3 mm to (109.9, 102.8), turned to 90 degrees
- moved RN3 99.2 mm to (119.2, 106.8), turned to -90 degrees
- moved C37 97.8 mm to (121.5, 126.8)
- moved C27 97.7 mm to (120.8, 118.4), turned to 180 degrees
- moved D1 97.0 mm to (103.8, 128.8)
- moved Y2 96.3 mm to (120.8, 116.5), turned to -90 degrees
- moved R19 96.3 mm to (107.2, 98.6), turned to 180 degrees
- moved C52 96.2 mm to (119.6, 126.8), turned to 0 degrees
- moved C28 96.1 mm to (119.1, 116.4)
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Connections:
- J3 pad 4: Net-(J3-Pin_4) -> +3V3
- U1 pad 14: /LED0 -> unconnected-(U1-PE17/CSI_D13/LCD_D19-Pad14)
Routing:
- net +1V2: track 0.00 -> 93.3 mm, vias 0 -> 11
- net +3V3: track 0.00 -> 76.4 mm, vias 0 -> 18
- net +5V: track 0.00 -> 29.0 mm, vias 0 -> 10
- net GND: track 0.00 -> 23.9 mm, vias 0 -> 85
- net +3V0: track 0.00 -> 21.4 mm, vias 0 -> 4
- net /UART0_TX: track 0.00 -> 18.4 mm, vias 0 -> 1
- net +1V8: track 0.00 -> 18.3 mm, vias 0 -> 4
- net /UART0_RX: track 0.00 -> 17.2 mm, vias 0 -> 1
- net SVREF: track 0.00 -> 14.1 mm, vias 0 -> 2
- net /LED_STLINK: track 0.00 -> 13.8 mm, vias 0 -> 1
- net /WL_UART_TX: track 0.00 -> 13.4 mm, vias 0 -> 1
- net /WL_UART_RX: track 0.00 -> 13.2 mm, vias 0 -> 1
- net /T_JTCK_SWCLK: track 0.00 -> 12.2 mm, vias 0 -> 1
- net /WL_SDIO_D3: track 0.00 -> 11.9 mm, vias 0 -> 1
- net /T_JTMS_SWDIO: track 0.00 -> 11.7 mm, vias 0 -> 1
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- added copper zone on F.Cu, net +1V2
- added copper zone on B.Cu, net +1V8
- added copper zone on F.Cu, net +1V8
- added copper zone on B.Cu, net +3V3
- added copper zone on F.Cu, net +3V3
- added copper zone on B.Cu, net +5V
- added copper zone on In2.Cu, net +5V
- added copper zone on B.Cu, net Net-(U2-LX1)
- added copper zone on B.Cu, net Net-(U2-LX2)
- added copper zone on B.Cu, net Net-(U2-LX3)
- added copper zone on F.Cu, net VBUS
Other:
- board size 20.5 x 41.1 mm -> 24.2 x 42.3 mm
- board text added: "F103CB"
- board text added: "Linux"
- board text added: "RM2026 ZZY"
- board text added: "TF Card"
- board text added: "TypeC"
- board text added: "V3S"
- board text added: "Wireless JLink"

Commit message: V2 Production
Parts:
- removed C40: 100nF, Capacitor_SMD:C_0402_1005Metric
- removed C48: 1uF, Capacitor_SMD:C_0402_1005Metric
- C34, C44, C51, R18, R19, R4: moved to B.Cu
- RN1, RN2: footprint Resistor_SMD:R_Array_Convex_4x0402 -> Resistor_SMD:R_Array_Convex_4x0603
- moved R4 10.1 mm to (118.8, 101.0), turned to 0 degrees
- moved C24 10.1 mm to (107.2, 101.8), turned to -90 degrees
- moved R18 9.35 mm to (118.8, 100.0), turned to 0 degrees
- moved C14 1.71 mm to (117.1, 101.1), turned to 180 degrees
- moved R19 1.30 mm to (105.9, 98.7), turned to -90 degrees
- moved C34 1.12 mm to (120.9, 110.1)
- moved RN2 1.04 mm to (103.0, 112.8)
- moved D2 1.00 mm to (107.2, 98.6), turned to 180 degrees
- moved C46 0.91 mm to (102.9, 120.0)
- moved C57 0.72 mm to (102.3, 115.2), turned to 180 degrees
- moved C35 0.30 mm to (118.6, 104.7)
- moved RN1 0.26 mm to (103.0, 117.6)
- moved C26 0.23 mm to (116.8, 98.1)
Connections:
- J3 pad 1: Net-(J3-Pin_1) -> +3V3
- J3 pad 2: Net-(J3-Pin_2) -> GND
- J3 pad 3: GND -> Net-(J3-Pin_3)
- J3 pad 4: +3V3 -> Net-(J3-Pin_4)
- R18 pad 2: Net-(J3-Pin_2) -> Net-(J3-Pin_3)
- R4 pad 2: Net-(J3-Pin_1) -> Net-(J3-Pin_4)
- RN2 pad 1: /WL_SDIO_D1 -> unconnected-(RN2-R1.1-Pad1)
- RN2 pad 2: /WL_SDIO_D0 -> /WL_SDIO_D1
- RN2 pad 3: /WL_SDIO_CLK -> /WL_SDIO_D0
- RN2 pad 6: unconnected-(RN2-R3.2-Pad6) -> +3V3
- RN2 pad 8: +3V3 -> unconnected-(RN2-R1.2-Pad8)
- U1 pad 39: /WL_UART_TX -> unconnected-(U1-PB0/UART2_TX/PB_EINT0-Pad39)
- U1 pad 40: /WL_UART_RX -> unconnected-(U1-PB1/UART2_RX/PB_EINT1-Pad40)
- U1 pad 45: unconnected-(U1-PB6/TWI0_SCK/PB_EINT6-Pad45) -> /TFT_DC
- U1 pad 46: unconnected-(U1-PB7/TWI0_SDA/PB_EINT7-Pad46) -> /TFT_RST
- U7 pad 42: /WL_UART_RX -> unconnected-(U7-UART_OUT-Pad42)
- U7 pad 43: /WL_UART_TX -> unconnected-(U7-UART_IN-Pad43)
Routing:
- net /WL_UART_TX: track 13.4 -> 0.00 mm, vias 1 -> 0
- net /TFT_RST: track 0.70 -> 14.0 mm, vias 1 -> 2
- net /WL_UART_RX: track 13.2 -> 0.00 mm, vias 1 -> 0
- net +3V0: track 21.4 -> 34.2 mm
- net /TFT_DC: track 0.10 -> 12.0 mm, vias 1 -> 2
- net +1V2: track 93.3 -> 104.5 mm, vias 11 -> 9
- net /ST_SWCLK: track 0.00 -> 10.6 mm
- net Net-(J3-Pin_3): track 0.00 -> 7.67 mm, vias 0 -> 1
- net /T_JTMS_SWDIO: track 11.7 -> 5.22 mm, vias 1 -> 0
- net /LED_STLINK: track 13.8 -> 20.1 mm
- net Net-(J3-Pin_4): track 0.00 -> 5.60 mm, vias 0 -> 1
- net +3V3: track 76.4 -> 80.9 mm, vias 18 -> 24
- net /SDC0_D0: track 6.93 -> 10.0 mm, vias 0 -> 1
- net Net-(J3-Pin_2): track 2.84 -> 0.00 mm
- net Net-(J3-Pin_1): track 2.74 -> 0.00 mm
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- added copper zone on In2.Cu, net +3V3
- added copper zone on B.Cu, net GND
- added copper zone on F.Cu, net GND
- added copper zone on In1.Cu, net GND
Other:
- board text added: "1"
- board text added: "12"
- board text added: "3GCD"
