File: Hardware/WirelessJLink_V3S.kicad_sch (KiCad schematic)
At the start: 147 parts, among them J1 Micro_SD_Card, J2 USB_C_Receptacle_USB2.0, J3 USB_C_Receptacle_USB2.0, J4 JLink_Upload, J5 JLINK_OUT, J6 24V_IN, Q1 S8050, SW1 海龟, U1 V831, U3 RS3236, U4 CH343P, U5 STM32F103CBT6, U6 W25Q128, U7 RTL8723BS, U8 RY8411, Y2 24MHz, Y3 8MHz

Commit message: V2 sch & layout Half Cplt
Parts:
- removed C13, C3, C72, C73: 10uF, Capacitor_SMD:C_1206_3216Metric, symbol Device:C
- removed C2: 10nF, Capacitor_SMD:C_0603_1608Metric, symbol Device:C
- removed C25: 10uF, Capacitor_SMD:C_0603_1608Metric, symbol Device:C
- removed C36, C69: 100nF, Capacitor_SMD:C_0603_1608Metric, symbol Device:C
- removed C70: 100nF, Resistor_SMD:R_0603_1608Metric, symbol Device:C
- removed C71: 20pF, Resistor_SMD:R_0603_1608Metric, symbol Device:C
- removed D3: K34, Diode_SMD:D_SMF, symbol Device:D
- removed F3: Fuse, Fuse:Fuse_1206_3216Metric, symbol Device:Fuse
- removed J3: USB_C_Receptacle_USB2.0, 0_RM2024:USB_C_Receptacle_HRO_TYPE-C-31-M-12_NO_HOLE, symbol Connector:USB_C_Receptacle_USB2.0
- removed J5: JLINK_OUT, Connector_Molex:Molex_PicoBlade_53261-0471_1x04-1MP_P1.25mm_Horizontal, symbol Connector_Generic_MountingPin:Conn_01x04_MountingPin
- removed J6: 24V_IN, Connector_AMASS:AMASS_XT30PW-M_1x02_P2.50mm_Horizontal, symbol Connector_Generic:Conn_01x02
- removed L4: 4.7uH, Inductor_SMD:L_Sunlord_SWPA252012S, symbol Device:L
- removed Q1: S8050, Package_TO_SOT_SMD:SOT-23, symbol Transistor_BJT:BC817
- removed R14, R15: 5.1K, Resistor_SMD:R_0603_1608Metric, symbol Device:R
- removed R16, R17: 33, Resistor_SMD:R_0603_1608Metric, symbol Device:R_Small
- removed R18: 100K, Resistor_SMD:R_0603_1608Metric, symbol Device:R_Small
- removed R2: 53.6K, Resistor_SMD:R_0603_1608Metric, symbol Device:R
- removed R20: 100R, Resistor_SMD:R_0603_1608Metric, symbol Device:R
- removed R21, R23, R33: 10K, Resistor_SMD:R_0603_1608Metric, symbol Device:R
- removed R22: 4.7K, Resistor_SMD:R_0603_1608Metric, symbol Device:R
- removed R26, R27, R3: 10k, Resistor_SMD:R_0603_1608Metric, symbol Device:R
- removed R28, R29: 33R, Resistor_SMD:R_0603_1608Metric, symbol Device:R
- removed R30: 1.5K, Resistor_SMD:R_0603_1608Metric, symbol Device:R
- removed R34: 36K, Resistor_SMD:R_0603_1608Metric, symbol Device:R
- removed R35, R41: 1K, Resistor_SMD:R_0603_1608Metric, symbol Device:R
- removed R36: 100, Resistor_SMD:R_0603_1608Metric, symbol Device:R
- removed R43: 33K, Resistor_SMD:R_0603_1608Metric, symbol Device:R
- removed SW1: 海龟, Button_Switch_SMD:SW_Push_1P1T_NO_CK_KMR2, symbol Switch:SW_Push
- removed U3: RS3236, Package_TO_SOT_SMD:SOT-23-5, symbol Regulator_Linear:LDK130-12_SOT23_SOT353
- removed U6: W25Q128, Package_SO:SOIC-8_5.23x5.23mm_P1.27mm, symbol Memory_Flash:W25Q128JVS
- removed U8: RY8411, Package_TO_SOT_SMD:SOT-23-6, symbol 0_RM2024:RY8411
- removed Y3: 8MHz, Crystal:Resonator_SMD_Murata_CSTxExxV-3Pin_3.0x1.1mm, symbol Device:Crystal_GND3
- added C13, C25, C3: 10uF, Capacitor_SMD:C_0402_1005Metric, symbol Device:C_Small
- added J3: JLink_Upload, Connector_Hirose:Hirose_DF13-04P-1.25DS_1x04_P1.25mm_Horizontal, symbol Connector_Generic:Conn_01x04
- added R18, R4: 33R, Resistor_SMD:R_0402_1005Metric, symbol Device:R
- added U6: HT7133, Package_TO_SOT_SMD:SOT-23-3, symbol Regulator_Linear:XC6206PxxxMR
- added Y1: 8MHz, Crystal:Resonator_SMD_Murata_CSTxExxV-3Pin_3.0x1.1mm, symbol Device:Crystal_GND3
- AE1: footprint 0_RM2024:IPXE4 -> RM2024:IPEX_1
- C1, C14, C15, C16, C17, C18, C19, C22, C23, C26, C27, C28, C29, C30, C31, C32, C33, C34, C35, C37, C38, C39, C40, C41, C42, C43, C44, C45, C46, C47, C48, C49, C50, C51, C52, C53, C54, C55, C56, C57, C58, C59, C60, C61, C62, C63, C64, C65, C66, C67, C68: footprint Capacitor_SMD:C_0603_1608Metric -> Capacitor_SMD:C_0402_1005Metric
- C10, C11, C12, C4, C5, C6: footprint Capacitor_SMD:C_1206_3216Metric -> Capacitor_SMD:C_0402_1005Metric
- C20, C21: value 20pF -> 100nF; footprint Capacitor_SMD:C_0603_1608Metric -> Capacitor_SMD:C_0402_1005Metric
- C24: value 100nF -> 10uF; footprint Capacitor_SMD:C_0603_1608Metric -> Capacitor_SMD:C_0805_2012Metric
- D2, D4: footprint LED_SMD:LED_0603_1608Metric -> LED_SMD:LED_0402_1005Metric
- J1: footprint 0_RM2024:TF_Card_Short2 -> RM2024:TF_Card_Short2
- J2: footprint 0_RM2024:USB_C_Receptacle_HRO_TYPE-C-31-M-12_NO_HOLE -> Connector_USB:USB_C_Receptacle_GCT_USB4110
- J4: footprint Connector_Molex:Molex_PicoBlade_53048-0410_1x04_P1.25mm_Horizontal -> RM2024:1.25Upload
- R1, R12, R13, R37, R38, R39, R40, R42, R44, R45, R46, R5: footprint Resistor_SMD:R_0603_1608Metric -> Resistor_SMD:R_0402_1005Metric
- R10: value 100K -> 10K
- R19: value 10K -> 1K; footprint Resistor_SMD:R_0603_1608Metric -> Resistor_SMD:R_0402_1005Metric
- R6: value 10K -> 200K
- R7: value 200K -> 10K
- R9: value 10K -> 100K
- RN1, RN2: footprint Resistor_SMD:R_Array_Convex_4x0603 -> Resistor_SMD:R_Array_Convex_4x0402
- U2: footprint Package_DFN_QFN:HVQFN-24-1EP_4x4mm_P0.5mm_EP2.6x2.6mm_ThermalVias -> Package_DFN_QFN:HVQFN-24-1EP_4x4mm_P0.5mm_EP2.6x2.6mm
- U7: footprint 0_RM2024:RTL8723BS -> RM2024:RTL8723BS
Connections:
- net OTG_DM is gone; now on net JLINK_DM: U1.110 (USB-DM)
- net OTG_DP is gone; now on net JLINK_DP: U1.111 (USB-DP)
- net T_SWDIO_IN is gone; now on net T_JTMS_SWDIO: U5.25 (PB12)
- net +1V2: now also C11.2, C8.2, L2.2, R7.1, C13.2; no longer C10.2, C7.2, L1.2, R6.1
- net +1V8: now also C10.2, C7.2, L1.2, R6.1, C3.2; no longer C11.2, C8.2, L2.2, R7.1
- net +3V0: now also U6.2 (VO)
- net +3V3: now also C20.1, C21.1, J4.1 (Pin_1), R19.2, U5.10 (PA0), U5.39 (PB3), C25.2; no longer J4.4 (Pin_4)
- net +5V: now also U6.3 (VI)
- net GND: now also C20.2, C21.2, J4.2 (Pin_2), U5.2 (PC13), U5.3 (PC14), U5.44 (BOOT0), C13.1, C25.1, C3.1, J3.3 (Pin_3), U6.1 (GND), Y1.2; no longer C20.1, C21.1, J4.3 (Pin_3), R19.2
- net JLINK_DXIN: now also Y1.3; no longer C20.2
- net JLINK_DXOUT: now also Y1.1; no longer C21.2
- net ST_SWCLK: now also J4.3 (Pin_3); no longer J4.2 (Pin_2)
- net ST_SWDIO: now also J4.4 (Pin_4); no longer J4.1 (Pin_1)
- net T_JTCK_SWCLK: now also R18.1
- net T_JTMS_SWDIO: now also R4.1
- net at F2.1: now also J3.4 (Pin_4)
- net at D2.2 (A): now also R19.1
- net JLINK_USB_RENUM: no longer names the net of U5.38 (PA15)
- new net: J3.1 (Pin_1), R4.2
- new net: J3.2 (Pin_2), R18.2
- no-connect marks 112 -> 111
Other:
- note added: "JLink"
- note removed: "FLASH"
- note removed: "JLINK"
- note removed: "PA2: TXD PA3: RXD PB13: SWCLK PB14: SWDIO PB0: NRST"
- moved on the sheet: C1, C10, C16, C17, C18, C26, C27, C28, C29, C30, C31, C33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

Commit message: V2 Hardware Half Cplt
Parts:
- removed C20, C21, C22: 100nF, Capacitor_SMD:C_0402_1005Metric, symbol Device:C
- removed C43, C47: 100nF, Capacitor_SMD:C_0402_1005Metric, symbol Device:C_Small
- removed C60: 1uF, Capacitor_SMD:C_0402_1005Metric, symbol Device:C_Small
- removed D4: LED, LED_SMD:LED_0402_1005Metric, symbol Device:LED
- removed F2: 1A, Fuse:Fuse_1206_3216Metric, symbol Device:Polyfuse
- removed R1: 1K, Resistor_SMD:R_0402_1005Metric, symbol Device:R
- added C2, C36, C69: 10uF, Capacitor_SMD:C_0402_1005Metric, symbol Device:C_Small
- added H1, H2, H3, H4: M2, MountingHole:MountingHole_2.2mm_M2_DIN965, symbol Mechanical:MountingHole
- added J5: TFT, RM2024:1.47TFT_12P, symbol Connector_Generic:Conn_01x12
- C1: value 100nF -> 10uF
Connections:
- net +1V2: now also C2.2
- net +3V3: now also J3.4 (Pin_4), C69.2, J5.10 (Pin_10), J5.9 (Pin_9)
- net +5V: now also C36.2
- net GND: now also C2.1, C36.1, C69.1, J5.1 (Pin_1), J5.11 (Pin_11), J5.12 (Pin_12), J5.8 (Pin_8)
- net SPI0_CLK: now also J5.4 (Pin_4)
- net SPI0_CS: now also J5.5 (Pin_5)
- net SPI0_MOSI: now also J5.3 (Pin_3)
- net LED0: no longer names the net of U1.14 (PE17/CSI_D13/LCD_D19)
- new net TFT_DC: J5.6 (Pin_6)
- new net TFT_RST: J5.2 (Pin_2)
- no-connect marks 111 -> 114
Other:
- moved on the sheet: C23, C24

Commit message: V2 Production
Parts:
- removed C40: 100nF, Capacitor_SMD:C_0402_1005Metric, symbol Device:C_Small
- removed C48: 1uF, Capacitor_SMD:C_0402_1005Metric, symbol Device:C_Small
- RN1, RN2: footprint Resistor_SMD:R_Array_Convex_4x0402 -> Resistor_SMD:R_Array_Convex_4x0603
Connections:
- net +3V3: now also J3.1 (Pin_1), RN2.6 (R3.2); no longer J3.4 (Pin_4), RN2.8 (R1.2)
- net GND: now also J3.2 (Pin_2); no longer J3.3 (Pin_3)
- net TFT_DC: now also U1.45 (PB6/TWI0_SCK/PB_EINT6)
- net TFT_RST: now also U1.46 (PB7/TWI0_SDA/PB_EINT7)
- net WL_SDIO_CLK: no longer RN2.3 (R3.1)
- net WL_SDIO_D0: now also RN2.3 (R3.1); no longer RN2.2 (R2.1)
- net WL_SDIO_D1: now also RN2.2 (R2.1); no longer RN2.1 (R1.1)
- net at R4.2: now also J3.4 (Pin_4); no longer J3.1 (Pin_1)
- net at R18.2: now also J3.3 (Pin_3); no longer J3.2 (Pin_2)
- net WL_UART_RX: no longer names the net of U1.40 (PB1/UART2_RX/PB_EINT1)
- net WL_UART_RX: no longer U7.42 (UART_OUT)
- net WL_UART_TX: no longer names the net of U1.39 (PB0/UART2_TX/PB_EINT0)
- net WL_UART_TX: no longer U7.43 (UART_IN)
- no-connect marks 114 -> 117
Other:
- moved on the sheet: RN1, RN2
